File: KiCAD/senior_design_gateway.kicad_pcb (KiCad board)
At the start: 2 copper layers, 159 x 109 mm, 9 parts

Commit message: edits by Eric during 2/21 meeting
Parts:
- moved CO2 32.1 mm to (176.4, 122.8)
Routing:
- net Net-(CO2-SDA): track 0.00 -> 91.8 mm
- net Net-(CO2-SCL): track 0.00 -> 89.1 mm
- net +5V: track 0.00 -> 34.5 mm
- added copper zone on B.Cu, net GND
Changed lines of the file:
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@@
     (fp_rect (start 0 0) (end 29.464 25.4)
       (stroke (width 0.1) (type default)) (fill none) (layer "F.SilkS"))
-    (pad "1" thru_hole circle (at 2.54 2.159 270) (size 1.524 1.524) (drill 0.762) (layers "*.Cu" "*.Mask")
+    (pad "1" thru_hole circle (at 2.54 2.159 270) (size 1.778 1.778) (drill 1.0922) (layers "*.Cu" "*.Mask")
       (net 12 "+3.3V") (pinfunction "Vin") (pintype "power_in"))
-    (pad "2" thru_hole circle (at 2.54 4.699 270) (size 1.524 1.524) (drill 0.762) (layers "*.Cu" "*.Mask")
+    (pad "2" thru_hole circle (at 2.54 4.699 270) (size 1.778 1.778) (drill 1.0922) (layers "*.Cu" "*.Mask")
       (net 4 "GND") (pinfunction "GND") (pintype "input"))
-    (pad "3" thru_hole circle (at 2.54 7.239 270) (size 1.524 1.524) (drill 0.762) (layers "*.Cu" "*.Mask")
+    (pad "3" thru_hole circle (at 2.54 7.239 270) (size 1.778 1.778) (drill 1.0922) (layers "*.Cu" "*.Mask")
       (net 13 "unconnected-(LoraWAN1-EN-Pad3)") (pinfunction "EN") (pintype "no_connect"))
-    (pad "4" thru_hole circle (at 2.54 9.779 270) (size 1.524 1.524) (drill 0.762) (layers "*.Cu" "*.Mask")
+    (pad "4" thru_hole circle (at 2.54 9.779 270) (size 1.778 1.778) (drill 1.0922) (layers "*.Cu" "*.Mask")
       (net 14 "Net-(ESP32-WROOM-32E1-SCK)") (pinfunction "SCK") (pintype "input"))
-    (pad "5" thru_hole circle (at 2.54 12.319 270) (size 1.524 1.524) (drill 0.762) (layers "*.Cu" "*.Mask")
+    (pad "5" thru_hole circle (at 2.54 12.319 270) (size 1.778 1.778) (drill 1.0922) (layers "*.Cu" "*.Mask")
       (net 15 "Net-(ESP32-WROOM-32E1-MISO)") (pinfunction "MISO") (pintype "input"))
-    (pad "6" thru_hole circle (at 2.54 14.859 270) (size 1.524 1.524) (drill 0.762) (layers "*.Cu" "*.Mask")
+    (pad "6" thru_hole circle (at 2.54 14.859 270) (size 1.778 1.778) (drill 1.0922) (layers "*.Cu" "*.Mask")
       (net 16 "Net-(ESP32-WROOM-32E1-MOSI)") (pinfunction "MOSI") (pintype "input"))
-    (pad "7" thru_hole circle (at 2.54 17.399 270) (size 1.524 1.524) (drill 0.762) (layers "*.Cu" "*.Mask")
+    (pad "7" thru_hole circle (at 2.54 17.399 270) (size 1.778 1.778) (drill 1.0922) (layers "*.Cu" "*.Mask")
       (net 17 "Net-(ESP32-WROOM-32E1-D04)") (pinfunction "CS") (pintype "input"))
-    (pad "8" thru_hole circle (at 2.54 19.939 270) (size 1.524 1.524) (drill 0.762) (layers "*.Cu" "*.Mask")
+    (pad "8" thru_hole circle (at 2.54 19.939 270) (size 1.778 1.778) (drill 1.0922) (layers "*.Cu" "*.Mask")
       (net 18 "Net-(ESP32-WROOM-32E1-D06)") (pinfunction "RST") (pintype "input"))
-    (pad "9" thru_hole circle (at 2.54 22.479 270) (size 1.524 1.524) (drill 0.762) (layers "*.Cu" "*.Mask"))
-    (pad "10" thru_hole circle (at 28.194 12.7 90) (size 1.524 1.524) (drill 0.762) (layers "*.Cu" "*.Mask"))
-    (pad "11" thru_hole circle (at 28.194 10.16 90) (size 1.524 1.524) (drill 0.762) (layers "*.Cu" "*.Mask"))
-    (pad "12" thru_hole circle (at 28.194 7.62 90) (size 1.524 1.524) (drill 0.762) (layers "*.Cu" "*.Mask"))
-    (pad "13" thru_hole circle (at 28.194 5.08 90) (size 1.524 1.524) (drill 0.762) (layers "*.Cu" "*.Mask"))
-    (pad "14" thru_hole circle (at 28.194 2.54 90) (size 1.524 1.524) (drill 0.762) (layers "*.Cu" "*.Mask"))
+    (pad "9" thru_hole circle (at 2.54 22.479 270) (size 1.778 1.778) (drill 1.0922) (layers "*.Cu" "*.Mask"))
+    (pad "10" thru_hole circle (at 28.194 12.7 270) (size 1.778 1.778) (drill 1.0922) (layers "*.Cu" "*.Mask"))
+    (pad "11" thru_hole circle (at 28.194 10.16 270) (size 1.778 1.778) (drill 1.0922) (layers "*.Cu" "*.Mask"))
+    (pad "12" thru_hole circle (at 28.194 7.62 270) (size 1.778 1.778) (drill 1.0922) (layers "*.Cu" "*.Mask"))
+    (pad "13" thru_hole circle (at 28.194 5.08 270) (size 1.778 1.778) (drill 1.0922) (layers "*.Cu" "*.Mask"))
+    (pad "14" thru_hole circle (at 28.194 2.54 270) (size 1.778 1.778) (drill 1.0922) (layers "*.Cu" "*.Mask"))
   )
   (footprint "Sensors:CO2" (layer "F.Cu")
-    (at 183.7325 91.54 -90)
+    (at 176.3665 122.782 -90)
     (property "Sheetfile" "senior_design_gateway.kicad_sch")
     (property "Sheetname" "")
@@
       (stroke (width 0.1) (type default)) (fill none) (layer "F.SilkS"))
     (dimension (type aligned) (layer "F.SilkS")
-      (pts (xy 163.4125 99.16) (xy 163.4125 101.7))
+      (pts (xy 156.0465 130.402) (xy 156.0465 132.942))
       (height -2.54)
-      (gr_text "0.1000 in" (at 164.8525 100.43 90) (layer "F.SilkS")
+      (gr_text "0.1000 in" (at 157.4865 131.672 90) (layer "F.SilkS")
         (effects (font (size 1 1) (thickness 0.1)))
       )
@@
   (gr_rect (start 50.8 50.8) (end 209.804 159.766)
     (stroke (width 0.1) (type default)) (fill none) (layer "Edge.Cuts"))
-  (gr_rect (start 58.42 58.42) (end 203.2 152.4)
-    (stroke (width 0.1) (type default)) (fill none) (layer "Margin"))
-  (dimension (type aligned) (layer "Edge.Cuts")
-    (pts (xy 209.804 50.8) (xy 50.8 50.8))
-    (height 5.079999)
-    (gr_text "6.2600 in" (at 130.302 44.570001) (layer "Edge.Cuts")
-      (effects (font (size 1 1) (thickness 0.15)))
-    )
-    (format (prefix "") (suffix "") (units 3) (units_format 1) (precision 4))
-    (style (thickness 0.1) (arrow_length 1.27) (text_position_mode 0) (extension_height 0.58642) (extension_offset 0.5) keep_text_aligned)
-  )
-  (dimension (type aligned) (layer "Edge.Cuts")
-    (pts (xy 209.804 50.8) (xy 209.804 159.766))
-    (height -6.096)
-    (gr_text "4.2900 in" (at 214.75 105.283 90) (layer "Edge.Cuts")
-      (effects (font (size 1 1) (thickness 0.15)))
-    )
-    (format (prefix "") (suffix "") (units 3) (units_format 1) (precision 4))
-    (style (thickness 0.1) (arrow_length 1.27) (text_position_mode 0) (extension_height 0.58642) (extension_offset 0.5) keep_text_aligned)
-  )
   (via (at 60.2996 59.7916) (size 4.572) (drill 4.4958) (layers "F.Cu" "B.Cu") (net 0))
   (via (at 200.3044 150.7744) (size 4.572) (drill 4.4958) (layers "F.Cu" "B.Cu") (net 0))
+  (segment (start 104.2305 123.9885) (end 105.41 122.809) (width 1.27) (layer "B.Cu") (net 1))
+  (segment (start 105.41 119.38) (end 105.41 114.3) (width 1.27) (layer "B.Cu") (net 1))
+  (segment (start 101.1031 123.9885) (end 104.2305 123.9885) (width 1.27) (layer "B.Cu") (net 1))
+  (segment (start 105.41 122.809) (end 105.41 119.38) (width 1.27) (layer "B.Cu") (net 1))
+  (segment (start 105.41 114.3) (end 105.41 99.3426) (width 1.27) (layer "B.Cu") (net 1))
+  (segment (start 105.41 99.3426) (end 109.8058 94.9468) (width 1.27) (layer "B.Cu") (net 1))
+  (segment (start 109.8058 87.3268) (end 116.078 93.599) (width 0.25) (layer "F.Cu") (net 2))
+  (segment (start 116.205 116.205) (end 113.03 119.38) (width 0.25) (layer "F.Cu") (net 2))
+  (segment (start 116.078 93.599) (end 116.078 116.078) (width 0.25) (layer "F.Cu") (net 2))
+  (segment (start 116.078 116.078) (end 116.205 116.205) (width 0.25) (layer "F.Cu") (net 2))
+  (segment (start 113.03 119.38) (end 113.03 122.301) (width 0.25) (layer "B.Cu") (net 2))
+  (segment (start 113.03 122.301) (end 129.54 138.811) (width 0.25) (layer "B.Cu") (net 2))
+  (segment (start 129.54 138.811) (end 152.908 138.811) (width 0.25) (layer "B.Cu") (net 2))
+  (segment (start 152.908 138.811) (end 153.697 138.022) (width 0.25) (layer "B.Cu") (net 2))
+  (segment (start 153.697 138.022) (end 156.0465 138.022) (width 0.25) (layer "B.Cu") (net 2))
+  (segment (start 109.8058 89.8668) (end 114.935 94.996) (width 0.25) (layer "F.Cu") (net 3))
+  (segment (start 114.935 112.395) (end 113.03 114.3) (width 0.25) (layer "F.Cu") (net 3))
+  (segment (start 114.935 94.996) (end 114.935 112.395) (width 0.25) (layer "F.Cu") (net 3))
+  (segment (start 109.22 123.063) (end 109.22 118.11) (width 0.25) (layer "B.Cu") (net 3))
+  (segment (start 109.22 118.11) (end 113.03 114.3) (width 0.25) (layer "B.Cu") (net 3))
+  (segment (start 156.0465 140.562) (end 126.719 140.562) (width 0.25) (layer "B.Cu") (net 3))
+  (segment (start 126.719 140.562) (end 109.22 123.063) (width 0.25) (layer "B.Cu") (net 3))
+  (zone (net 4) (net_name "GND") (layer "B.Cu") (hatch edge 0.5)
+    (connect_pads (clearance 0.5))
+    (min_thickness 0.25) (filled_areas_thickness no)
+    (fill yes (thermal_gap 0.5) (thermal_bridge_width 0.5))
+    (polygon
+      (pts
+        (xy 43.18 48.26)
+        (xy 213.36 48.26)
+        (xy 213.36 165.1)
+        (xy 43.18 165.1)
+      )
+    )
+  )
 )
