File: KiCAD/senior_design_gateway.kicad_sch (KiCad schematic)
At the start: 9 parts

Commit message: edits by Eric during 2/21 meeting
Parts:
- added TP1: TestPoint, TestPoint:TestPoint_Loop_D2.54mm_Drill1.5mm_Beaded, symbol Connector:TestPoint
- R1: value R -> 4.7k
Connections:
- net GND: now also TP1.1
- net at CO2.5 (SDA), R2.2, SEN55.3 (SDA): now also ESP32-WROOM-32E1.1 (SDA); no longer ESP32-WROOM-32E1. (Vin)
Changed lines of the file:
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@@
     (pin "")
     (pin "")
-    (pin "")
+    (pin "1")
     (instances
       (project "senior_design_gateway"
@@
       (effects (font (size 1.27 1.27)) (justify left))
     )
-    (property "Value" "R" (at 86.36 63.5 0)
-      (effects (font (size 1.27 1.27)) (justify left) hide)
+    (property "Value" "4.7k" (at 86.36 63.5 0)
+      (effects (font (size 1.27 1.27)) (justify left))
     )
     (property "Footprint" "Resistor_THT:R_Axial_DIN0207_L6.3mm_D2.5mm_P7.62mm_Horizontal" (at 76.962 67.31 90)
@@
     )
   )
+  (symbol (lib_id "power:GND") (at 208.28 140.335 0) (unit 1)
+    (in_bom yes) (on_board yes) (dnp no) (fields_autoplaced)
+    (property "Reference" "#PWR015" (at 208.28 146.685 0)
+      (effects (font (size 1.27 1.27)) hide)
+    )
+    (property "Value" "GND" (at 208.28 145.415 0)
+      (effects (font (size 1.27 1.27)))
+    )
+    (property "Footprint" "" (at 208.28 140.335 0)
+      (effects (font (size 1.27 1.27)) hide)
+    )
+    (property "Datasheet" "" (at 208.28 140.335 0)
+      (effects (font (size 1.27 1.27)) hide)
+    )
+    (pin "1")
+    (instances
+      (project "senior_design_gateway"
+        (path "/7aefded4-b51d-417d-a9e8-a87f1079445b"
+          (reference "#PWR015") (unit 1)
+        )
+      )
+    )
+  )
   (symbol (lib_id "power:GND") (at 181.61 53.34 0) (unit 1)
     (in_bom yes) (on_board yes) (dnp no) (fields_autoplaced)
@@
         )
       )
+    )
+  )
+  (symbol (lib_id "Connector:TestPoint") (at 208.28 140.335 0) (unit 1)
+    (in_bom yes) (on_board yes) (dnp no) (fields_autoplaced)
+    (property "Reference" "TP1" (at 210.82 135.763 0)
+      (effects (font (size 1.27 1.27)) (justify left))
+    )
+    (property "Value" "TestPoint" (at 210.82 138.303 0)
+      (effects (font (size 1.27 1.27)) (justify left))
+    )
+    (property "Footprint" "TestPoint:TestPoint_Loop_D2.54mm_Drill1.5mm_Beaded" (at 213.36 140.335 0)
+      (effects (font (size 1.27 1.27)) hide)
+    )
+    (property "Datasheet" "~" (at 213.36 140.335 0)
+      (effects (font (size 1.27 1.27)) hide)
+    )
+    (pin "1")
+    (instances
+      (project "senior_design_gateway"
+        (path "/7aefded4-b51d-417d-a9e8-a87f1079445b"
+          (reference "TP1") (unit 1)
+        )
+      )
